File: hardware/project/EVTPS65130.kicad_sch (KiCad schematic)
At the start: 53 parts, among them J1 USB_C_Receptacle_PowerOnly_6P, J2 Conn_01x04_Pin, Q10 PMOS, U3 TPS65130RGE

Commit message: Updated PCB
Connections:
- net GND is gone; now on net AGND: C27.2, C28.2, C29.2, C30.2, C31.2, C32.2, C33.2, C34.2, C35.2, C41.2, C42.2, C43.2, C44.2, C45.2, C46.2, C47.2, C48.2, C49.2, D1.1 (K), D2.1 (K), D3.2 (A), J1.A12 (GND), J1.B12 (GND), J1.SH (SHIELD), J2.2 (Pin_2), J2.3 (Pin_3), L2.1, R69.2, R70.1, U3.2 (PGND), U3.25 (EP), U3.3 (PGND)
- net -12V_OUT: now reaches C47.1, C49.1, D9.2 (A), FB2.1, R63.2, R64.2, U3.15 (VNEG)
- net +12V_OUT: now reaches C40.1, C46.1, C48.1, D8.1 (K), FB1.1, R60.2, U3.23 (VPOS)
Changed lines of the file:
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@@
 	(wire
 		(pts
+			(xy 35.56 149.86) (xy 43.18 149.86)
+		)
+		(stroke
+			(width 0)
+			(type default)
+		)
+	)
+	(wire
+		(pts
 			(xy 212.09 83.82) (xy 212.09 86.36)
 		)
@@
 	(wire
 		(pts
+			(xy 43.18 149.86) (xy 43.18 151.13)
+		)
+		(stroke
+			(width 0)
+			(type default)
+		)
+	)
+	(wire
+		(pts
 			(xy 191.77 133.35) (xy 199.39 133.35)
 		)
@@
 	(wire
 		(pts
+			(xy 35.56 151.13) (xy 35.56 149.86)
+		)
+		(stroke
+			(width 0)
+			(type default)
+		)
+	)
+	(wire
+		(pts
 			(xy 113.03 53.34) (xy 113.03 55.88)
 		)
@@
 		)
 	)
+	(label "+12V_OUT"
+		(at 156.21 73.66 0)
+		(effects
+			(font
+				(size 1.27 1.27)
+			)
+			(justify left bottom)
+		)
+	)
+	(label "-12V_OUT"
+		(at 180.34 133.35 0)
+		(effects
+			(font
+				(size 1.27 1.27)
+			)
+			(justify left bottom)
+		)
+	)
 	(symbol
 		(lib_id "Device:C")
@@
 	(symbol
 		(lib_id "power:GND")
+		(at 43.18 151.13 0)
+		(unit 1)
+		(body_style 1)
+		(exclude_from_sim no)
+		(in_bom yes)
+		(on_board yes)
+		(in_pos_files yes)
+		(dnp no)
+		(fields_autoplaced yes)
+		(property "Reference" "#PWR097"
+			(at 43.18 157.48 0)
+			(hide yes)
+			(show_name no)
+			(do_not_autoplace no)
+			(effects
+				(font
+					(size 1.27 1.27)
+				)
+			)
+		)
+		(property "Value" "GND"
+			(at 43.18 156.21 0)
+			(hide yes)
+			(show_name no)
+			(do_not_autoplace no)
+			(effects
+				(font
+					(size 1.27 1.27)
+				)
+			)
+		)
+		(property "Footprint" ""
+			(at 43.18 151.13 0)
+			(hide yes)
+			(show_name no)
+			(do_not_autoplace no)
+			(effects
+				(font
+					(size 1.27 1.27)
+				)
+			)
+		)
+		(property "Datasheet" ""
+			(at 43.18 151.13 0)
+			(hide yes)
+			(show_name no)
+			(do_not_autoplace no)
+			(effects
+				(font
+					(size 1.27 1.27)
+				)
+			)
+		)
+		(property "Description" "Power symbol creates a global label with name \"GND\" , ground"
+			(at 43.18 151.13 0)
+			(hide yes)
+			(show_name no)
+			(do_not_autoplace no)
+			(effects
+				(font
+					(size 1.27 1.27)
+				)
+			)
+		)
+		(pin "1"
+		)
+		(instances
+			(project "EVTPS65130"
+				(path "/b1cb391d-ea8e-4faa-bb90-2b0ee6abebaa"
+					(reference "#PWR097")
+					(unit 1)
+				)
+			)
+		)
+	)
+	(symbol
+		(lib_id "power:GND")
 		(at 137.16 151.13 0)
 		(unit 1)
@@
 					(unit 1)
 				)
+			)
+		)
+	)
+	(symbol
+		(lib_id "power:GND")
+		(at 35.56 151.13 0)
+		(unit 1)
+		(body_style 1)
+		(exclude_from_sim no)
+		(in_bom yes)
+		(on_board yes)
+		(in_pos_files yes)
+		(dnp no)
+		(property "Reference" "#PWR096"
+			(at 35.56 157.48 0)
+			(hide yes)
+			(show_name no)
+			(do_not_autoplace no)
+			(effects
+				(font
+					(size 1.27 1.27)
+				)
+			)
+		)
+		(property "Value" "AGND"
+			(at 35.56 154.94 0)
+			(show_name no)
+			(do_not_autoplace no)
+			(effects
+				(font
+					(size 1.27 1.27)
+				)
+			)
+		)
+		(property "Footprint" ""
+			(at 35.56 151.13 0)
+			(hide yes)
+			(show_name no)
+			(do_not_autoplace no)
+			(effects
+				(font
+					(size 1.27 1.27)
+				)
+			)
+		)
+		(property "Datasheet" ""
+			(at 35.56 151.13 0)
+			(hide yes)
+			(show_name no)
+			(do_not_autoplace no)
+			(effects
+				(font
+					(size 1.27 1.27)
+				)
+			)
+		)
+		(property "Description" "Power symbol creates a global label with name \"GND\" , ground"
+			(at 35.56 151.13 0)
+			(hide yes)
+			(show_name no)
+			(do_not_autoplace no)
+			(effects
+				(font
+					(size 1.27 1.27)
+				)
+			)
+		)
+		(pin "1"
+		)
+		(instances
+			(project "EVTPS65130"
+				(path "/b1cb391d-ea8e-4faa-bb90-2b0ee6abebaa"
+					(reference "#PWR096")
+					(unit 1)
+				)

Commit message: Finished PCB
Parts:
- removed J2: Conn_01x04_Pin, Connector_PinHeader_2.54mm:PinHeader_1x04_P2.54mm_Vertical, symbol Connector:Conn_01x04_Pin
- added C50, C51, C52, C53: 100n, Capacitor_SMD:C_0402_1005Metric, symbol Device:C
- added D4: LED, LED_SMD:LED_0603_1608Metric, symbol Device:LED
- added J2: Conn_01x06_Pin, Connector_PinHeader_2.54mm:PinHeader_1x06_P2.54mm_Vertical, symbol Connector:Conn_01x06_Pin
- added R71: 680R, Resistor_SMD:R_0402_1005Metric, symbol Device:R_US
- added U1: L78L33_SOT89, Package_TO_SOT_SMD:SOT-89-3, symbol Regulator_Linear:L78L33_SOT89
Connections:
- net AGND: now also C50.2, C51.2, C52.2, C53.2, D4.1 (K), J2.3 (Pin_3), J2.4 (Pin_4), U1.2 (GND)
- net VDD: now also J2.1 (Pin_1)
- net VIN: now also C50.1, C51.1, C52.1, J2.5 (Pin_5), U1.3 (IN)
- net VSS: now also J2.6 (Pin_6)
- new net: D4.2 (A), R71.1
- new net +3.3V: C53.1, J2.2 (Pin_2), R71.2, U1.1 (OUT)
